File: 32a4u.sch (EAGLE design)
At the start: 11 parts

Commit message: tweak traces, standardize labeling
Connections:
- net GND: now also U$3.1, U$3.17, U$3.2, U$4.3
- net VUSB: no longer U$3.17, U$4.3

Commit message: LED on PE2
Parts:
- added LED1: (no value), microbuilder:LED0603
- added R1: (no value), nonolith:RESISTOR0603
Connections:
- new net N$1: LED1.C, R1.1
- net GND: now also R1.2
- net PE2: now also LED1.A
Other:
- moved on the sheet: U$4
Changed lines of the file:
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@@
 <part name="C3" library="nonolith" deviceset="CAP_CERAMIC" device="0603"/>
 <part name="C4" library="nonolith" deviceset="CAP_CERAMIC" device="0603"/>
+<part name="LED1" library="microbuilder" deviceset="LED" device="0603"/>
+<part name="U$1" library="nonolith" deviceset="GND" device=""/>
+<part name="U$5" library="nonolith" deviceset="GND" device=""/>
+<part name="U$6" library="nonolith" deviceset="GND" device=""/>
+<part name="R1" library="nonolith" deviceset="RESISTOR" device="0603"/>
 </parts>
 <sheets>
@@
 <instance part="U$2" gate="G$1" x="127" y="0" rot="R180"/>
 <instance part="U$3" gate="G$1" x="-35.56" y="63.5"/>
-<instance part="U$4" gate="G$1" x="111.76" y="63.5" rot="R180"/>
+<instance part="U$4" gate="G$1" x="121.92" y="66.04" rot="R180"/>
 <instance part="C1" gate="G$1" x="91.44" y="25.4"/>
 <instance part="C2" gate="G$1" x="99.06" y="25.4"/>
@@
 <instance part="C3" gate="G$1" x="-5.08" y="10.16"/>
 <instance part="C4" gate="G$1" x="0" y="5.08"/>
+<instance part="LED1" gate="G$1" x="91.44" y="48.26" rot="R270"/>
+<instance part="U$1" gate="G$1" x="101.6" y="40.64"/>
+<instance part="U$5" gate="G$1" x="5.08" y="0"/>
+<instance part="U$6" gate="G$1" x="99.06" y="15.24"/>
+<instance part="R1" gate="G$1" x="96.52" y="43.18"/>
 </instances>
 <busses>
@@
 </segment>
 <segment>
-<wire x1="101.6" y1="83.82" x2="99.06" y2="83.82" width="0" layer="91"/>
-<label x="96.52" y="83.82" size="1.778" layer="95"/>
+<wire x1="111.76" y1="86.36" x2="109.22" y2="86.36" width="0" layer="91"/>
+<label x="106.68" y="86.36" size="1.778" layer="95"/>
 <pinref part="U$4" gate="G$1" pin="2"/>
 </segment>
@@
 <pinref part="C1" gate="G$1" pin="P$2"/>
 <pinref part="C2" gate="G$1" pin="P$2"/>
+<pinref part="U$6" gate="G$1" pin="GND"/>
+<junction x="99.06" y="17.78"/>
 </segment>
 <segment>
@@
 </segment>
 <segment>
-<wire x1="101.6" y1="86.36" x2="99.06" y2="86.36" width="0" layer="91"/>
-<label x="96.52" y="86.36" size="1.778" layer="95"/>
+<wire x1="111.76" y1="88.9" x2="109.22" y2="88.9" width="0" layer="91"/>
+<label x="106.68" y="88.9" size="1.778" layer="95"/>
 <pinref part="U$4" gate="G$1" pin="1"/>
 </segment>
@@
 <label x="5.08" y="2.54" size="1.778" layer="95"/>
 <junction x="0" y="2.54"/>
-</segment>
-<segment>
-<wire x1="101.6" y1="81.28" x2="99.06" y2="81.28" width="0" layer="91"/>
-<label x="96.52" y="81.28" size="1.778" layer="95"/>
+<pinref part="U$5" gate="G$1" pin="GND"/>
+</segment>
+<segment>
+<wire x1="111.76" y1="83.82" x2="109.22" y2="83.82" width="0" layer="91"/>
+<label x="106.68" y="83.82" size="1.778" layer="95"/>
 <pinref part="U$4" gate="G$1" pin="3"/>
 </segment>
@@
 <label x="-22.86" y="40.64" size="1.778" layer="95"/>
 </segment>
+<segment>
+<pinref part="R1" gate="G$1" pin="2"/>
+<pinref part="U$1" gate="G$1" pin="GND"/>
+</segment>
 </net>
 <net name="PDI-DATA" class="0">
@@
 </segment>
 <segment>
-<wire x1="101.6" y1="40.64" x2="99.06" y2="40.64" width="0" layer="91"/>
-<label x="96.52" y="40.64" size="1.778" layer="95"/>
+<wire x1="111.76" y1="43.18" x2="109.22" y2="43.18" width="0" layer="91"/>
+<label x="106.68" y="43.18" size="1.778" layer="95"/>
 <pinref part="U$4" gate="G$1" pin="19"/>
 </segment>
@@
 </segment>
 <segment>
-<wire x1="101.6" y1="43.18" x2="99.06" y2="43.18" width="0" layer="91"/>
-<label x="96.52" y="43.18" size="1.778" layer="95"/>
+<wire x1="111.76" y1="45.72" x2="109.22" y2="45.72" width="0" layer="91"/>
+<label x="106.68" y="45.72" size="1.778" layer="95"/>
 <pinref part="U$4" gate="G$1" pin="18"/>
 </segment>
@@
 </segment>
 <segment>
-<wire x1="101.6" y1="45.72" x2="99.06" y2="45.72" width="0" layer="91"/>
-<label x="96.52" y="45.72" size="1.778" layer="95"/>
+<wire x1="111.76" y1="48.26" x2="109.22" y2="48.26" width="0" layer="91"/>
+<label x="106.68" y="48.26" size="1.778" layer="95"/>
 <pinref part="U$4" gate="G$1" pin="17"/>
 </segment>
@@
 </segment>
 <segment>
-<wire x1="101.6" y1="48.26" x2="99.06" y2="48.26" width="0" layer="91"/>
-<label x="96.52" y="48.26" size="1.778" layer="95"/>
+<wire x1="111.76" y1="50.8" x2="109.22" y2="50.8" width="0" layer="91"/>
+<label x="106.68" y="50.8" size="1.778" layer="95"/>
 <pinref part="U$4" gate="G$1" pin="16"/>
 </segment>
@@
 </segment>
 <segment>
-<wire x1="101.6" y1="50.8" x2="99.06" y2="50.8" width="0" layer="91"/>
-<label x="96.52" y="50.8" size="1.778" layer="95"/>
+<wire x1="111.76" y1="53.34" x2="109.22" y2="53.34" width="0" layer="91"/>
+<label x="106.68" y="53.34" size="1.778" layer="95"/>
 <pinref part="U$4" gate="G$1" pin="15"/>
 </segment>
@@
 </segment>
 <segment>
-<wire x1="101.6" y1="53.34" x2="99.06" y2="53.34" width="0" layer="91"/>
-<label x="96.52" y="53.34" size="1.778" layer="95"/>
+<wire x1="111.76" y1="55.88" x2="109.22" y2="55.88" width="0" layer="91"/>
+<label x="106.68" y="55.88" size="1.778" layer="95"/>
 <pinref part="U$4" gate="G$1" pin="14"/>
 </segment>
@@
 </segment>
 <segment>
-<wire x1="101.6" y1="55.88" x2="99.06" y2="55.88" width="0" layer="91"/>
-<label x="96.52" y="55.88" size="1.778" layer="95"/>
+<wire x1="111.76" y1="58.42" x2="109.22" y2="58.42" width="0" layer="91"/>
+<label x="106.68" y="58.42" size="1.778" layer="95"/>
 <pinref part="U$4" gate="G$1" pin="13"/>
 </segment>
@@
 </segment>
 <segment>
-<wire x1="101.6" y1="58.42" x2="99.06" y2="58.42" width="0" layer="91"/>
-<label x="96.52" y="58.42" size="1.778" layer="95"/>
+<wire x1="111.76" y1="60.96" x2="109.22" y2="60.96" width="0" layer="91"/>
+<label x="106.68" y="60.96" size="1.778" layer="95"/>
 <pinref part="U$4" gate="G$1" pin="12"/>
 </segment>
@@
 </segment>
 <segment>
-<wire x1="101.6" y1="60.96" x2="99.06" y2="60.96" width="0" layer="91"/>
-<label x="96.52" y="60.96" size="1.778" layer="95"/>
+<wire x1="111.76" y1="63.5" x2="109.22" y2="63.5" width="0" layer="91"/>
+<label x="106.68" y="63.5" size="1.778" layer="95"/>
 <pinref part="U$4" gate="G$1" pin="11"/>
 </segment>
@@
 </segment>
 <segment>
-<wire x1="101.6" y1="63.5" x2="99.06" y2="63.5" width="0" layer="91"/>
-<label x="96.52" y="63.5" size="1.778" layer="95"/>
+<wire x1="111.76" y1="66.04" x2="109.22" y2="66.04" width="0" layer="91"/>
+<label x="106.68" y="66.04" size="1.778" layer="95"/>
 <pinref part="U$4" gate="G$1" pin="10"/>
 </segment>
@@
 </segment>
 <segment>
-<wire x1="101.6" y1="66.04" x2="99.06" y2="66.04" width="0" layer="91"/>
-<label x="96.52" y="66.04" size="1.778" layer="95"/>
+<wire x1="111.76" y1="68.58" x2="109.22" y2="68.58" width="0" layer="91"/>
+<label x="106.68" y="68.58" size="1.778" layer="95"/>
 <pinref part="U$4" gate="G$1" pin="9"/>
 </segment>
@@
 </segment>
 <segment>
-<wire x1="101.6" y1="68.58" x2="99.06" y2="68.58" width="0" layer="91"/>
-<label x="96.52" y="68.58" size="1.778" layer="95"/>
+<wire x1="111.76" y1="71.12" x2="109.22" y2="71.12" width="0" layer="91"/>
+<label x="106.68" y="71.12" size="1.778" layer="95"/>
 <pinref part="U$4" gate="G$1" pin="8"/>
 </segment>
@@
 </segment>
 <segment>
-<wire x1="101.6" y1="71.12" x2="96.52" y2="71.12" width="0" layer="91"/>
-<label x="96.52" y="71.12" size="1.778" layer="95"/>
+<wire x1="111.76" y1="73.66" x2="106.68" y2="73.66" width="0" layer="91"/>
+<label x="106.68" y="73.66" size="1.778" layer="95"/>
 <pinref part="U$4" gate="G$1" pin="7"/>
 </segment>
@@
 </segment>
 <segment>
-<wire x1="101.6" y1="73.66" x2="99.06" y2="73.66" width="0" layer="91"/>
-<label x="96.52" y="73.66" size="1.778" layer="95"/>
+<wire x1="111.76" y1="76.2" x2="109.22" y2="76.2" width="0" layer="91"/>
+<label x="106.68" y="76.2" size="1.778" layer="95"/>
 <pinref part="U$4" gate="G$1" pin="6"/>
 </segment>
@@
 <label x="83.82" y="53.34" size="1.778" layer="95"/>
 <pinref part="ATXMEGA32A4U" gate="G$1" pin="RXD0/OC0C/PE2"/>
-</segment>
-<segment>
-<wire x1="101.6" y1="76.2" x2="99.06" y2="76.2" width="0" layer="91"/>
-<label x="96.52" y="76.2" size="1.778" layer="95"/>
+<pinref part="LED1" gate="G$1" pin="A"/>
+<wire x1="86.36" y1="53.34" x2="91.44" y2="53.34" width="0.1524" layer="91"/>
+</segment>
+<segment>
+<wire x1="111.76" y1="78.74" x2="109.22" y2="78.74" width="0" layer="91"/>
+<label x="106.68" y="78.74" size="1.778" layer="95"/>
 <pinref part="U$4" gate="G$1" pin="5"/>
 </segment>
@@
 </segment>
 <segment>
-<wire x1="101.6" y1="78.74" x2="99.06" y2="78.74" width="0" layer="91"/>
-<label x="96.52" y="78.74" size="1.778" layer="95"/>
+<wire x1="111.76" y1="81.28" x2="109.22" y2="81.28" width="0" layer="91"/>
+<label x="106.68" y="81.28" size="1.778" layer="95"/>
 <pinref part="U$4" gate="G$1" pin="4"/>
 </segment>
@@
 </segment>
 </net>
+<net name="N$1" class="0">
+<segment>
+<pinref part="LED1" gate="G$1" pin="C"/>
+<pinref part="R1" gate="G$1" pin="1"/>
+<wire x1="91.44" y1="43.18" x2="91.44" y2="45.72" width="0.1524" layer="91"/>
+</segment>
+</net>

Commit message: routed 5v0 rail to headers, added pair of decoupling capacitors
Parts:
- added C5, C6: (no value), nonolith:CAP_CERAMIC0603
Connections:
- net GND: now also C5.P$2, C6.P$1; no longer U$3.1, U$3.19
- net VUSB: now also C5.P$1, C6.P$2, U$3.1, U$3.19
Changed lines of the file:
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@@
 <?xml version="1.0" encoding="utf-8"?>
 <!DOCTYPE eagle SYSTEM "eagle.dtd">
-<eagle version="6.1">
+<eagle version="6.3">
 <drawing>
 <settings>
@@
 <part name="U$6" library="nonolith" deviceset="GND" device=""/>
 <part name="R1" library="nonolith" deviceset="RESISTOR" device="0603"/>
+<part name="C5" library="nonolith" deviceset="CAP_CERAMIC" device="0603"/>
+<part name="C6" library="nonolith" deviceset="CAP_CERAMIC" device="0603"/>
 </parts>
 <sheets>
@@
 <instance part="U$6" gate="G$1" x="99.06" y="15.24"/>
 <instance part="R1" gate="G$1" x="96.52" y="43.18"/>
+<instance part="C5" gate="G$1" x="-7.62" y="81.28"/>
+<instance part="C6" gate="G$1" x="-7.62" y="43.18"/>
 </instances>
 <busses>
@@
 <label x="147.32" y="63.5" size="1.778" layer="95"/>
 <pinref part="CN1" gate="G$1" pin="VBUS"/>
+</segment>
+<segment>
+<label x="-20.32" y="86.36" size="1.778" layer="95"/>
+<pinref part="U$3" gate="G$1" pin="19"/>
+<pinref part="C5" gate="G$1" pin="P$1"/>
+<wire x1="-7.62" y1="86.36" x2="-25.4" y2="86.36" width="0" layer="91"/>
+</segment>
+<segment>
+<pinref part="U$3" gate="G$1" pin="1"/>
+<label x="-22.86" y="40.64" size="1.778" layer="95"/>
+<pinref part="C6" gate="G$1" pin="P$2"/>
+<wire x1="-25.4" y1="40.64" x2="-7.62" y2="40.64" width="0" layer="91"/>
 </segment>
 </net>
@@
 </segment>
 <segment>
-<wire x1="-25.4" y1="86.36" x2="-20.32" y2="86.36" width="0" layer="91"/>
-<label x="-20.32" y="86.36" size="1.778" layer="95"/>
-<pinref part="U$3" gate="G$1" pin="19"/>
-</segment>
-<segment>
 <wire x1="111.76" y1="88.9" x2="109.22" y2="88.9" width="0" layer="91"/>
 <label x="106.68" y="88.9" size="1.778" layer="95"/>
@@
 </segment>
 <segment>
-<pinref part="U$3" gate="G$1" pin="1"/>
-<wire x1="-25.4" y1="40.64" x2="-22.86" y2="40.64" width="0" layer="91"/>
-<label x="-22.86" y="40.64" size="1.778" layer="95"/>
-</segment>
-<segment>
 <pinref part="R1" gate="G$1" pin="2"/>
 <pinref part="U$1" gate="G$1" pin="GND"/>
 </segment>
+<segment>
+<pinref part="C5" gate="G$1" pin="P$2"/>
+<pinref part="C6" gate="G$1" pin="P$1"/>
+<wire x1="-7.62" y1="78.74" x2="-7.62" y2="63.5" width="0" layer="91"/>
+<wire x1="-7.62" y1="63.5" x2="-7.62" y2="48.26" width="0" layer="91"/>
+<wire x1="-7.62" y1="63.5" x2="-2.54" y2="63.5" width="0" layer="91"/>
+<label x="-5.08" y="63.5" size="1.778" layer="95"/>
+</segment>
 </net>
