File: 32a4u.brd (EAGLE design)
At the start: 29.2 x 49.5 mm, 11 parts

Commit message: LED on PE2
Parts:
- added LED1: (no value), microbuilder:CHIPLED_0603
- added R1: (no value), nonolith:0603
- moved C1 2.16 mm to (11.0, 15.5), turned to 180 degrees
Connections:
- new net N$1: LED1.C, R1.1
- net GND: now also R1.2
- net PE2: now also LED1.A
Routing:
- net VCC: track 81.8 -> 86.5 mm, vias 0 -> 1
- net GND: track 5.69 -> 9.36 mm, vias 17 -> 18
- net PE2: track 15.0 -> 12.6 mm, vias 1 -> 0
- net PE3: track 14.3 -> 16.6 mm, vias 1 -> 0
- net N$1: track 0.00 -> 2.18 mm
Changed lines of the file:
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@@
 <element name="U$3" library="SparkFun" package="1X19" value="M19" x="29.845" y="3.175" smashed="yes" rot="R90"/>
 <element name="U$4" library="SparkFun" package="1X19" value="M19" x="4.445" y="3.175" smashed="yes" rot="R90"/>
-<element name="C1" library="nonolith" package="0603" value="" x="9.652" y="13.843" smashed="yes" rot="R90">
-<attribute name="NAME" x="11.303" y="13.716" size="0.762" layer="25" font="vector" ratio="12" rot="R90"/>
-<attribute name="VALUE" x="10.287" y="15.621" size="0.4064" layer="27" font="vector" rot="R90"/>
+<element name="C1" library="nonolith" package="0603" value="" x="11.049" y="15.494" smashed="yes" rot="R180">
+<attribute name="NAME" x="9.906" y="16.637" size="0.762" layer="25" font="vector" ratio="12"/>
+<attribute name="VALUE" x="9.271" y="16.129" size="0.4064" layer="27" font="vector" rot="R180"/>
 </element>
 <element name="C2" library="nonolith" package="0603" value="" x="17.145" y="35.814" smashed="yes" rot="R180">
-<attribute name="NAME" x="15.367" y="35.56" size="0.762" layer="25" font="vector" ratio="12" rot="R180"/>
+<attribute name="NAME" x="18.669" y="34.544" size="0.762" layer="25" font="vector" ratio="12" rot="R180"/>
 </element>
 <element name="CN1" library="nonolith" package="USB-MICROB" value="" x="17.272" y="49.276" rot="R180"/>
@@
 <element name="C4" library="nonolith" package="0603" value="" x="23.876" y="12.954" smashed="yes">
 <attribute name="NAME" x="24.13" y="14.224" size="0.762" layer="25" font="vector" ratio="12"/>
+</element>
+<element name="LED1" library="microbuilder" package="CHIPLED_0603" value="" x="10.668" y="13.208" rot="R270"/>
+<element name="R1" library="nonolith" package="0603" value="" x="10.922" y="11.176" smashed="yes" rot="R180">
+<attribute name="NAME" x="12.446" y="9.906" size="0.762" layer="25" font="vector" ratio="10" rot="R180"/>
 </element>
 </elements>
@@
 <wire x1="18.3388" y1="24.892" x2="18.3388" y2="27.4828" width="0.254" layer="1"/>
 <wire x1="17.5419125" y1="19.8628" x2="14.776190625" y2="17.097078125" width="0.254" layer="1"/>
-<wire x1="14.776190625" y1="17.097078125" x2="10.6721125" y2="12.993" width="0.254" layer="1"/>
-<wire x1="10.6721125" y1="12.993" x2="9.652" y2="12.993" width="0.254" layer="1"/>
-<wire x1="4.445" y1="5.715" x2="9.652" y2="10.922" width="0.254" layer="1"/>
-<wire x1="9.652" y1="10.922" x2="9.652" y2="12.993" width="0.254" layer="1"/>
 <wire x1="15.494" y1="3.048" x2="14.224" y2="4.318" width="0.254" layer="16"/>
 <wire x1="14.224" y1="4.318" x2="6.096" y2="4.318" width="0.254" layer="16"/>
@@
 <vertex x="18.796" y="21.336"/>
 <vertex x="20.32" y="19.812"/>
-<vertex x="19.812" y="19.304"/>
-<vertex x="17.272" y="19.304"/>
-<vertex x="15.24" y="21.59"/>
-<vertex x="15.24" y="23.368"/>
-<vertex x="13.716" y="24.892"/>
+<vertex x="20.066" y="19.558"/>
+<vertex x="17.272" y="19.558"/>
+<vertex x="14.224" y="22.606"/>
+<vertex x="14.224" y="23.368"/>
+<vertex x="13.208" y="24.384"/>
+<vertex x="13.208" y="24.892"/>
 <vertex x="16.764" y="24.892"/>
 <vertex x="16.764" y="28.956"/>
@@
 <wire x1="18.095" y1="37.689" x2="26.761" y2="46.355" width="0.254" layer="1"/>
 <wire x1="26.761" y1="46.355" x2="29.845" y2="46.355" width="0.254" layer="1"/>
+<wire x1="14.776190625" y1="17.097078125" x2="13.1731125" y2="15.494" width="0.254" layer="1"/>
+<wire x1="11.899" y1="15.494" x2="11.684" y2="15.494" width="0.254" layer="1"/>
+<wire x1="13.1731125" y1="15.494" x2="11.899" y2="15.494" width="0.254" layer="1"/>
+<wire x1="14.224" y1="4.318" x2="14.224" y2="16.51" width="0.254" layer="16"/>
+<wire x1="14.224" y1="16.51" x2="17.526" y2="19.812" width="0.254" layer="16"/>
+<via x="17.526" y="19.812" extent="1-16" drill="0.3302"/>
+<wire x1="17.526" y1="19.812" x2="17.272" y2="20.066" width="0.254" layer="1"/>
 </signal>
 <signal name="VUSB">
@@
 <contactref element="JP1" pad="6"/>
 <via x="12.7" y="23.114" extent="1-16" drill="0.3302"/>
-<via x="14.224" y="13.716" extent="1-16" drill="0.3302"/>
+<via x="7.62" y="12.192" extent="1-16" drill="0.3302"/>
 <via x="19.558" y="44.704" extent="1-16" drill="0.3302"/>
 <contactref element="U$4" pad="3"/>
@@
 <via x="17.526" y="18.288" extent="1-16" drill="0.3302"/>
 <via x="16.002" y="32.766" extent="1-16" drill="0.3302"/>
+<wire x1="20.574" y1="18.288" x2="19.812" y2="19.05" width="0.254" layer="1"/>
+<wire x1="19.812" y1="19.05" x2="18.288" y2="19.05" width="0.254" layer="1"/>
+<wire x1="18.288" y1="19.05" x2="17.526" y2="18.288" width="0.254" layer="1"/>
+<contactref element="R1" pad="2"/>
+<via x="7.62" y="14.986" extent="1-16" drill="0.3302"/>
 </signal>
 <signal name="PDI-DATA">
@@
 <contactref element="ATXMEGA32A4U" pad="29"/>
 <contactref element="U$4" pad="6"/>
-<wire x1="13.3096" y1="18.1864" x2="13.6144" y2="18.1864" width="0.2032" layer="1"/>
-<wire x1="4.6736" y1="16.1036" x2="11.51996875" y2="16.1036" width="0.254" layer="1"/>
-<wire x1="13.6144" y1="18.1864" x2="13.64481875" y2="18.22845" width="0.2032" layer="1"/>
-<wire x1="4.445" y1="15.875" x2="4.6736" y2="16.1036" width="0.254" layer="1"/>
-<wire x1="11.51996875" y1="16.1036" x2="13.64481875" y2="18.22845" width="0.254" layer="1"/>
+<wire x1="13.64481875" y1="18.22845" x2="12.43436875" y2="17.018" width="0.254" layer="1"/>
+<wire x1="12.43436875" y1="17.018" x2="6.35" y2="17.018" width="0.254" layer="1"/>
+<wire x1="6.35" y1="17.018" x2="5.207" y2="15.875" width="0.254" layer="1"/>
+<wire x1="5.207" y1="15.875" x2="4.445" y2="15.875" width="0.254" layer="1"/>
 </signal>
 <signal name="PE2">
 <contactref element="ATXMEGA32A4U" pad="32"/>
 <contactref element="U$4" pad="5"/>
-<wire x1="15.494" y1="16.5608" x2="15.3924" y2="16.5608" width="0.2032" layer="1"/>
-<wire x1="16.3576" y1="17.4244" x2="15.494" y2="16.5608" width="0.254" layer="1"/>
-<wire x1="8.8392" y1="17.4244" x2="16.3576" y2="17.4244" width="0.254" layer="16"/>
-<wire x1="4.7752" y1="13.3604" x2="8.8392" y2="17.4244" width="0.254" layer="16"/>
-<wire x1="4.4704" y1="13.3604" x2="4.7752" y2="13.3604" width="0.2032" layer="16"/>
-<wire x1="15.3924" y1="16.5608" x2="15.341875" y2="16.53139375" width="0.2032" layer="1"/>
-<wire x1="4.445" y1="13.335" x2="4.4704" y2="13.3604" width="0.254" layer="16"/>
-<via x="16.3576" y="17.4244" extent="1-16" drill="0.3302"/>
+<contactref element="LED1" pad="A"/>
+<wire x1="15.341875" y1="16.53139375" x2="13.03448125" y2="14.224" width="0.254" layer="1"/>
+<wire x1="9.918" y1="13.208" x2="10.045" y2="13.335" width="0.254" layer="1"/>
+<wire x1="10.045" y1="13.335" x2="4.445" y2="13.335" width="0.254" layer="1"/>
+<wire x1="13.03448125" y1="14.224" x2="10.934" y2="14.224" width="0.254" layer="1"/>
+<wire x1="10.934" y1="14.224" x2="9.918" y2="13.208" width="0.254" layer="1"/>
 </signal>
 <signal name="PE3">
 <contactref element="ATXMEGA32A4U" pad="33"/>
 <contactref element="U$4" pad="4"/>
-<wire x1="15.9004" y1="14.7828" x2="15.9004" y2="15.9512" width="0.2032" layer="1"/>
-<wire x1="8.7376" y1="14.7828" x2="15.9004" y2="14.7828" width="0.254" layer="16"/>
-<wire x1="4.7752" y1="10.8204" x2="8.7376" y2="14.7828" width="0.254" layer="16"/>
-<wire x1="4.4704" y1="10.8204" x2="4.7752" y2="10.8204" width="0.2032" layer="16"/>
-<wire x1="15.9004" y1="15.9512" x2="15.9075625" y2="15.96570625" width="0.2032" layer="1"/>
-<wire x1="4.445" y1="10.795" x2="4.4704" y2="10.8204" width="0.2032" layer="16"/>
-<via x="15.9004" y="14.7828" extent="1-16" drill="0.3302"/>
+<wire x1="4.445" y1="10.795" x2="4.572" y2="10.668" width="0.254" layer="1"/>
+<wire x1="15.9075625" y1="15.9075625" x2="15.9075625" y2="15.96570625" width="0.254" layer="1"/>
+<wire x1="4.572" y1="10.668" x2="7.112" y2="10.668" width="0.254" layer="1"/>
+<wire x1="7.112" y1="10.668" x2="8.382" y2="9.398" width="0.254" layer="1"/>
+<wire x1="8.382" y1="9.398" x2="12.192" y2="9.398" width="0.254" layer="1"/>
+<wire x1="12.192" y1="9.398" x2="13.462" y2="10.668" width="0.254" layer="1"/>
+<wire x1="13.462" y1="10.668" x2="13.462" y2="13.462" width="0.254" layer="1"/>
+<wire x1="13.462" y1="13.462" x2="15.748" y2="15.748" width="0.254" layer="1"/>
+<wire x1="15.748" y1="15.748" x2="15.748" y2="16.002" width="0.254" layer="1"/>
+<wire x1="15.9075625" y1="15.96570625" x2="15.78429375" y2="15.96570625" width="0.254" layer="1"/>
+<wire x1="15.78429375" y1="15.96570625" x2="15.748" y2="16.002" width="0.254" layer="1"/>
 </signal>
 <signal name="PR0">
@@
 <wire x1="23.7141125" y1="26.035" x2="29.845" y2="26.035" width="0.254" layer="1"/>
 </signal>
+<signal name="N$1">
+<contactref element="LED1" pad="C"/>
+<contactref element="R1" pad="1"/>
+<wire x1="11.418" y1="13.208" x2="11.772" y2="12.854" width="0.254" layer="1"/>
+<wire x1="11.772" y1="12.854" x2="11.772" y2="11.176" width="0.254" layer="1"/>
+</signal>
 </signals>

Commit message: routed 5v0 rail to headers, added pair of decoupling capacitors
Parts:
- added C5, C6: (no value), nonolith:0603
Connections:
- net GND: now also C5.2, C6.1; no longer U$3.1, U$3.19
- net VUSB: now also C5.1, C6.2, U$3.1, U$3.19
Routing:
- net VUSB: track 7.28 -> 81.3 mm
- net VCC: track 86.5 -> 92.3 mm
Other:
- board text added: "5V"
Changed lines of the file:
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@@
 <?xml version="1.0" encoding="utf-8"?>
 <!DOCTYPE eagle SYSTEM "eagle.dtd">
-<eagle version="6.1">
+<eagle version="6.3">
 <drawing>
 <settings>
@@
 <text x="25.654" y="15.621" size="0.762" layer="25" font="vector" ratio="12">PA3</text>
 <text x="25.654" y="18.288" size="0.762" layer="25" font="vector" ratio="12">PA4</text>
-<text x="25.908" y="48.768" size="0.762" layer="25" font="vector" ratio="12">GND</text>
+<text x="25.908" y="48.768" size="0.762" layer="25" font="vector" ratio="12">5V</text>
 <text x="25.908" y="46.101" size="0.762" layer="25" font="vector" ratio="12">3.3V</text>
 <text x="25.654" y="40.767" size="0.762" layer="25" font="vector" ratio="12">PC1</text>
@@
 <text x="6.223" y="8.001" size="0.762" layer="25" font="vector" ratio="12">GND</text>
 <text x="26.289" y="5.207" size="0.762" layer="25" font="vector" ratio="12">GND</text>
-<text x="26.289" y="2.921" size="0.762" layer="25" font="vector" ratio="12">GND</text>
+<text x="26.289" y="2.921" size="0.762" layer="25" font="vector" ratio="12">5V</text>
 <text x="25.654" y="43.434" size="0.762" layer="25" font="vector" ratio="12">GND</text>
 </plain>
@@
 </class>
 </classes>
-<designrules>
+<designrules name="default">
 <description language="de">&lt;b&gt;EAGLE Design Rules&lt;/b&gt;
 &lt;p&gt;
@@
 <attribute name="NAME" x="12.446" y="9.906" size="0.762" layer="25" font="vector" ratio="10" rot="R180"/>
 </element>
+<element name="C5" library="nonolith" package="0603" value="" x="21.844" y="40.894" rot="R270"/>
+<element name="C6" library="nonolith" package="0603" value="" x="22.606" y="4.064"/>
 </elements>
 <signals>
@@
 <wire x1="17.995" y1="35.814" x2="17.907" y2="35.902" width="0.254" layer="1"/>
 <wire x1="17.907" y1="35.902" x2="17.907" y2="35.941" width="0.254" layer="1"/>
-<wire x1="18.095" y1="37.689" x2="26.761" y2="46.355" width="0.254" layer="1"/>
 <wire x1="26.761" y1="46.355" x2="29.845" y2="46.355" width="0.254" layer="1"/>
 <wire x1="14.776190625" y1="17.097078125" x2="13.1731125" y2="15.494" width="0.254" layer="1"/>
@@
 <via x="17.526" y="19.812" extent="1-16" drill="0.3302"/>
 <wire x1="17.526" y1="19.812" x2="17.272" y2="20.066" width="0.254" layer="1"/>
+<wire x1="18.095" y1="37.689" x2="18.252" y2="37.846" width="0.4064" layer="1"/>
+<wire x1="18.252" y1="37.846" x2="22.86" y2="37.846" width="0.4064" layer="1"/>
+<wire x1="22.86" y1="37.846" x2="24.638" y2="39.624" width="0.4064" layer="1"/>
+<wire x1="24.638" y1="39.624" x2="24.638" y2="44.196" width="0.4064" layer="1"/>
+<wire x1="24.638" y1="44.196" x2="26.797" y2="46.355" width="0.4064" layer="1"/>
+<wire x1="26.797" y1="46.355" x2="29.845" y2="46.355" width="0.4064" layer="1"/>
 </signal>
 <signal name="VUSB">
 <contactref element="U$2" pad="VIN"/>
 <contactref element="CN1" pad="P1"/>
-<wire x1="18.572" y1="46.601" x2="18.572" y2="41.686" width="0.254" layer="1"/>
+<wire x1="18.572" y1="46.601" x2="18.572" y2="42.418" width="0.254" layer="1"/>
+<wire x1="18.572" y1="42.418" x2="18.572" y2="41.686" width="0.254" layer="1"/>
 <wire x1="18.572" y1="41.686" x2="17.272" y2="40.386" width="0.254" layer="1"/>
 <wire x1="17.272" y1="40.386" x2="17.018" y2="40.132" width="0.254" layer="1"/>
 <wire x1="17.145" y1="40.289" x2="17.242" y2="40.386" width="0.254" layer="1"/>
 <wire x1="17.242" y1="40.386" x2="17.272" y2="40.386" width="0.254" layer="1"/>
+<contactref element="U$3" pad="19"/>
+<contactref element="U$3" pad="1"/>
+<wire x1="29.845" y1="48.895" x2="26.543" y2="48.895" width="0.4064" layer="1"/>
+<wire x1="26.543" y1="48.895" x2="21.717" y2="44.069" width="0.4064" layer="1"/>
+<wire x1="21.717" y1="44.069" x2="20.066" y2="42.418" width="0.4064" layer="1"/>
+<wire x1="20.066" y1="42.418" x2="18.572" y2="42.418" width="0.4064" layer="1"/>
+<wire x1="29.845" y1="3.175" x2="24.638" y2="8.382" width="0.4064" layer="16"/>
+<wire x1="24.638" y1="8.382" x2="24.638" y2="44.45" width="0.4064" layer="16"/>
+<wire x1="24.638" y1="44.45" x2="28.702" y2="48.514" width="0.4064" layer="16"/>
+<wire x1="28.702" y1="48.514" x2="29.718" y2="48.514" width="0.4064" layer="16"/>
+<contactref element="C5" pad="1"/>
+<contactref element="C6" pad="2"/>
+<wire x1="21.844" y1="41.744" x2="21.717" y2="41.871" width="0.4064" layer="1"/>
+<wire x1="21.717" y1="41.871" x2="21.717" y2="44.069" width="0.4064" layer="1"/>
+<wire x1="23.456" y1="4.064" x2="25.234" y2="2.286" width="0.4064" layer="1"/>
+<wire x1="25.234" y1="2.286" x2="27.94" y2="2.286" width="0.4064" layer="1"/>
+<wire x1="27.94" y1="2.286" x2="28.829" y2="3.175" width="0.4064" layer="1"/>
+<wire x1="28.829" y1="3.175" x2="29.845" y2="3.175" width="0.4064" layer="1"/>
+<wire x1="29.718" y1="48.514" x2="29.845" y2="48.895" width="0" layer="19" extent="16-16"/>
 </signal>
 <signal name="GND">
@@
 <contactref element="C1" pad="2"/>
 <contactref element="C2" pad="2"/>
-<contactref element="U$3" pad="19"/>
 <contactref element="U$4" pad="1"/>
 <via x="25.4" y="11.176" extent="1-16" drill="0.3302"/>
@@
 <contactref element="U$3" pad="17"/>
 <contactref element="U$3" pad="2"/>
-<contactref element="U$3" pad="1"/>
 <via x="19.812" y="14.224" extent="1-16" drill="0.3302"/>
 <via x="21.336" y="12.192" extent="1-16" drill="0.3302"/>
@@
 <contactref element="R1" pad="2"/>
 <via x="7.62" y="14.986" extent="1-16" drill="0.3302"/>
+<contactref element="C5" pad="2"/>
+<contactref element="C6" pad="1"/>
 </signal>
 <signal name="PDI-DATA">

Commit message: 10mil isolate on polygons
Routing:
- net GND: track 9.36 -> 15.6 mm
- net VUSB: track 81.3 -> 81.8 mm
Changed lines of the file:
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@@
 <?xml version="1.0" encoding="utf-8"?>
 <!DOCTYPE eagle SYSTEM "eagle.dtd">
-<eagle version="6.3">
+<eagle version="6.1">
 <drawing>
 <settings>
@@
 </class>
 </classes>
-<designrules name="default">
+<designrules>
 <description language="de">&lt;b&gt;EAGLE Design Rules&lt;/b&gt;
 &lt;p&gt;
@@
 <param name="mvStopFrame" value="1"/>
 <param name="mvCreamFrame" value="0"/>
-<param name="mlMinStopFrame" value="20mil"/>
+<param name="mlMinStopFrame" value="2mil"/>
 <param name="mlMaxStopFrame" value="2mil"/>
 <param name="mlMinCreamFrame" value="0mil"/>
@@
 <wire x1="13.0556" y1="24.9936" x2="13.1572" y2="24.892" width="0.254" layer="1"/>
 <wire x1="13.1572" y1="24.892" x2="18.3388" y2="24.892" width="0.254" layer="1"/>
-<polygon width="0.254" layer="1">
+<polygon width="0.254" layer="1" isolate="0.254">
 <vertex x="17.272" y="28.956"/>
 <vertex x="18.034" y="27.94"/>
@@
 <wire x1="24.638" y1="8.382" x2="24.638" y2="44.45" width="0.4064" layer="16"/>
 <wire x1="24.638" y1="44.45" x2="28.702" y2="48.514" width="0.4064" layer="16"/>
-<wire x1="28.702" y1="48.514" x2="29.718" y2="48.514" width="0.4064" layer="16"/>
+<wire x1="28.702" y1="48.514" x2="29.845" y2="48.514" width="0.4064" layer="16"/>
 <contactref element="C5" pad="1"/>
 <contactref element="C6" pad="2"/>
@@
 <wire x1="27.94" y1="2.286" x2="28.829" y2="3.175" width="0.4064" layer="1"/>
 <wire x1="28.829" y1="3.175" x2="29.845" y2="3.175" width="0.4064" layer="1"/>
-<wire x1="29.718" y1="48.514" x2="29.845" y2="48.895" width="0" layer="19" extent="16-16"/>
+<wire x1="29.845" y1="48.514" x2="29.845" y2="48.895" width="0.4064" layer="16"/>
 </signal>
 <signal name="GND">
@@
 <via x="15.24" y="44.704" extent="1-16" drill="0.3302"/>
 <via x="10.668" y="27.432" extent="1-16" drill="0.3302"/>
-<polygon width="0.4064" layer="16">
+<polygon width="0.4064" layer="16" isolate="0.254">
 <vertex x="-0.508" y="52.832"/>
 <vertex x="-0.508" y="-0.127"/>
@@
 <vertex x="36.83" y="53.467"/>
 </polygon>
-<polygon width="0.4064" layer="1" rank="5">
+<polygon width="0.4064" layer="1" isolate="0.254" rank="5">
 <vertex x="38.481" y="54.737"/>
 <vertex x="-2.413" y="54.737"/>
@@
 <contactref element="C5" pad="2"/>
 <contactref element="C6" pad="1"/>
+<wire x1="15.972" y1="46.601" x2="16.002" y2="46.601" width="0.4064" layer="1"/>
+<wire x1="16.002" y1="46.601" x2="16.002" y2="44.704" width="0.4064" layer="1"/>
+<wire x1="16.002" y1="44.704" x2="15.24" y2="44.704" width="0.4064" layer="1"/>
+<wire x1="9.398" y1="16.51" x2="12.954" y2="16.51" width="0.254" layer="1"/>
 </signal>
 <signal name="PDI-DATA">
